File: stepdriver_hw/Glidertrack.sch (KiCad schematic (older format))
At the start: 26 parts

Commit message: HW: start to trace pcb.
Parts:
- added C15, C16, C17: C, CAP_0603, symbol C
- added D1: DIODE, ~, symbol DIODE
- added D2, D3, D4: LED, ~, symbol LED
- added DA3: LD1117, ~, symbol LD1117
- added F1: FUSE0R, ~, symbol FUSE0R
- added R6, R7, R8: R, RES_0603, symbol R
- added XL3, XL5, XL7: CONN_3, ~, symbol CONN_3
- added XL4: CONN_2, ~, symbol CONN_2
- added XL6: CONN_10, ~, symbol CONN_10
- added XL8: BARREL_SOCKET, ~, symbol BARREL_SOCKET
- added XL?: CONN_16, ~, symbol CONN_16
- gave numbers to parts that had none: 26
Connections:
- net labels added: +VS, GPIOB10, GPIOB11, GPIOB12, GPIOB13, GPIOB14, GPIOB15, GPIOB3, GPIOB4, GPIOB5, GPIOB6, GPIOB7, GPIOB8, GPIOB9, MOTOR_BUSY, MOTOR_FLAG, MOTOR_SPI_CS, MOTOR_SPI_MISO, MOTOR_SPI_MOSI, MOTOR_SPI_SCK, MOTOR_STBY, MOTOR_STCK, WIFI_BOOT, WIFI_RESET
- net labels removed: SPI_MISO, SPI_MOSI, SPI_SCK
- wire segments 88 -> 190
- no-connect marks 2 -> 27
Other:
- moved on the sheet: C1, C10, C11, C12, C13, C14, C2, C3, C4, C5, C6, C7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

Commit message: HW: component placed.
Parts:
- removed XL?: CONN_16, ~, symbol CONN_16
- added C?: 0.1u, CAP_0603, symbol C
- added DA?: EEPROM_SPI, symbol EEPROM_SPI
- added R10, R9: 22K, RES_0603, symbol R
- added XL9: CONN_8, ~, symbol CONN_8
- C10, C9: value C -> 15p
- C15: value C -> 0.1u
- C16: value C -> 10u
- R5: value R -> 1K2
- R6, R7, R8: value R -> 22R
- XTAL1: value CRYSTAL -> 8/16 MHz
- renumbered D3 to LINK_UP1, D2 to POWER_UP1, D4 to RUN1
Connections:
- net labels added: EE_CK, EE_CS, EE_HOLD, EE_MISO, EE_MOSI, EE_SCK, EE_WRITE
- net labels removed: GPIOB10, GPIOB11, GPIOB12, GPIOB13, GPIOB14, GPIOB15
- wire segments 190 -> 196
Other:
- moved on the sheet: C1, C10, C17, C2, C3, C4, C5, C6, C7, C8, C9, DD1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

Commit message: HW: added MOSFET transistor on power WiFi module.
Parts:
- added Q1: IRLML6302, ~, symbol IRLML6302
- added R11: 10K, RES_0603, symbol R
- gave numbers to parts that had none: 2
Connections:
- net labels added: WIFI_PWR
- wire segments 196 -> 201
Other:
- moved on the sheet: C17, LINK_UP1, MDL1, POWER_UP1, R10, R6, R7, R8, R9, RUN1

Commit message: HW: PCB design proceed.
Parts:
- added HOLE1, HOLE2: HOLE_METALLED, symbol HOLE_METALLED
Connections:
- net labels added: PWR
- net labels removed: GPIOB3
- wire segments 201 -> 204
Other:
- moved on the sheet: Q1, R11
Changed lines of the file:
@@
 Sheet 1 1
 Title "Glidertrack"
-Date "11 dec 2014"
+Date "30 dec 2014"
 Rev ""
 Comp ""
@@
 	12800 2300 12950 2300
 Wire Wire Line
-	12800 1700 12800 2300
-Wire Wire Line
-	12500 1800 12500 1700
-Connection ~ 12500 1700
+	12800 1200 12800 2300
+Wire Wire Line
+	12500 1200 12500 1800
 $Comp
 L +3.3V #PWR024
 U 1 1 5481E4D5
-P 10950 1700
-F 0 "#PWR024" H 10950 1660 30  0001 C CNN
-F 1 "+3.3V" H 11030 1730 30  0000 C CNN
-F 2 "~" H 10950 1700 60  0000 C CNN
-F 3 "~" H 10950 1700 60  0000 C CNN
-	1    10950 1700
+P 10950 1200
+F 0 "#PWR024" H 10950 1160 30  0001 C CNN
+F 1 "+3.3V" H 11030 1230 30  0000 C CNN
+F 2 "~" H 10950 1200 60  0000 C CNN
+F 3 "~" H 10950 1200 60  0000 C CNN
+	1    10950 1200
 	-1   0    0    1
 $EndComp
@@
 Wire Wire Line
 	6550 3200 6700 3200
-Text Label 6550 2000 2    60   ~ 0
-GPIOB3
 Text Label 6550 2100 2    60   ~ 0
 GPIOB4
@@
 Wire Wire Line
 	3000 4800 3650 4800
-Text Label 3150 4100 0    60   ~ 0
-GPIOB3
 Text Label 3150 4200 0    60   ~ 0
 GPIOB4
@@
 Wire Wire Line
 	11950 1800 11950 1700
-Connection ~ 11950 1700
 Wire Wire Line
 	12150 1800 12150 1700
-Connection ~ 12150 1700
 Wire Wire Line
 	11950 2300 11950 2600
@@
 L IRLML6302 Q1
 U 1 1 5489849E
-P 11500 1750
-F 0 "Q1" H 11700 1800 60  0000 C CNN
-F 1 "IRLML6302" H 11900 1650 60  0000 C CNN
-F 2 "~" H 11500 1750 60  0000 C CNN
-F 3 "~" H 11500 1750 60  0000 C CNN
-	1    11500 1750
+P 11500 1250
+F 0 "Q1" H 11700 1300 60  0000 C CNN
+F 1 "IRLML6302" H 11900 1150 60  0000 C CNN
+F 2 "~" H 11500 1250 60  0000 C CNN
+F 3 "~" H 11500 1250 60  0000 C CNN
+	1    11500 1250
 	0    -1   -1   0
 $EndComp
 Wire Wire Line
-	10950 1700 11300 1700
-Wire Wire Line
-	11450 2300 11450 1950
-Wire Wire Line
-	11700 1700 12800 1700
+	10950 1200 11300 1200
+Wire Wire Line
+	11450 1800 11450 1450
+Wire Wire Line
+	11700 1200 12800 1200
 $Comp
 L R R11
 U 1 1 5489895C
-P 11050 2000
-F 0 "R11" V 11130 1850 50  0000 C CNN
-F 1 "10K" V 11050 2000 50  0000 C CNN
-F 2 "RES_0603" V 11130 2100 28  0000 C CNN
-F 3 "~" H 11050 2000 60  0000 C CNN
-	1    11050 2000
-	1    0    0    -1
-$EndComp
-Wire Wire Line
-	11050 1750 11050 1700
-Connection ~ 11050 1700
-Wire Wire Line
-	10850 2300 11450 2300
-Wire Wire Line
-	11050 2300 11050 2250
-Connection ~ 11050 2300
-Text Label 10850 2300 2    60   ~ 0
+P 11050 1500
+F 0 "R11" V 11130 1350 50  0000 C CNN
+F 1 "10K" V 11050 1500 50  0000 C CNN
+F 2 "RES_0603" V 11130 1600 28  0000 C CNN
+F 3 "~" H 11050 1500 60  0000 C CNN
+	1    11050 1500
+	1    0    0    -1
+$EndComp
+Wire Wire Line
+	11050 1250 11050 1200
+Connection ~ 11050 1200
+Wire Wire Line
+	10850 1800 11450 1800
+Wire Wire Line
+	11050 1800 11050 1750
+Connection ~ 11050 1800
+Text Label 10850 1800 2    60   ~ 0
 WIFI_PWR
 $Comp
 L PWR_FLAG #FLG052
 U 1 1 54898D30
+P 12800 1200
+F 0 "#FLG052" H 12800 1470 30  0001 C CNN
+F 1 "PWR_FLAG" H 12800 1430 30  0000 C CNN
+F 2 "~" H 12800 1200 60  0000 C CNN
+F 3 "~" H 12800 1200 60  0000 C CNN
+	1    12800 1200
+	1    0    0    -1
+$EndComp
+$Comp
+L +3.3V #PWR053
+U 1 1 5489910E
+P 3150 4100
+F 0 "#PWR053" H 3150 4060 30  0001 C CNN
+F 1 "+3.3V" H 3230 4130 30  0000 C CNN
+F 2 "~" H 3150 4100 60  0000 C CNN
+F 3 "~" H 3150 4100 60  0000 C CNN
+	1    3150 4100
+	1    0    0    -1
+$EndComp
+Text Label 6550 2000 2    60   ~ 0
+WIFI_PWR
+$Comp
+L HOLE_METALLED HOLE1
+U 1 1 5492EBC9
+P 9800 9950
+F 0 "HOLE1" H 9300 9900 60  0000 C CNN
+F 1 "HOLE_METALLED" H 9250 10000 60  0000 C CNN
+F 2 "" H 9800 9950 60  0000 C CNN
+F 3 "" H 9800 9950 60  0000 C CNN
+	1    9800 9950
+	0    1    1    0
+$EndComp
+$Comp
+L HOLE_METALLED HOLE2
+U 1 1 5492EBD8
+P 10050 9950
+F 0 "HOLE2" H 9550 9900 60  0000 C CNN
+F 1 "HOLE_METALLED" H 9500 10000 60  0000 C CNN
+F 2 "" H 10050 9950 60  0000 C CNN
+F 3 "" H 10050 9950 60  0000 C CNN
+	1    10050 9950
+	0    1    1    0
+$EndComp
+Wire Wire Line
+	9800 10250 9800 10500
+Wire Wire Line
+	9800 10500 10050 10500
+Wire Wire Line
+	10050 10250 10050 10600
+Connection ~ 10050 10500
+$Comp
+L GND #PWR054
+U 1 1 5492EEE5
+P 10050 10600
+F 0 "#PWR054" H 10140 10580 30  0001 C CNN
+F 1 "GND" H 10050 10520 30  0001 C CNN
+F 2 "~" H 10050 10600 60  0000 C CNN
+F 3 "~" H 10050 10600 60  0000 C CNN
+	1    10050 10600
+	1    0    0    -1
+$EndComp
+Connection ~ 12500 1200
+$Comp
+L +3.3V #PWR055
+U 1 1 54A2A8A6
+P 12150 1700
+F 0 "#PWR055" H 12150 1660 30  0001 C CNN
+F 1 "+3.3V" H 12230 1730 30  0000 C CNN
+F 2 "~" H 12150 1700 60  0000 C CNN
+F 3 "~" H 12150 1700 60  0000 C CNN
+	1    12150 1700
+	0    -1   -1   0
+$EndComp
+$Comp
+L +3.3V #PWR056
+U 1 1 54A2A8B5
 P 11950 1700
-F 0 "#FLG052" H 11950 1970 30  0001 C CNN
-F 1 "PWR_FLAG" H 11950 1930 30  0000 C CNN
+F 0 "#PWR056" H 11950 1660 30  0001 C CNN
+F 1 "+3.3V" H 12030 1730 30  0000 C CNN
 F 2 "~" H 11950 1700 60  0000 C CNN
 F 3 "~" H 11950 1700 60  0000 C CNN
 	1    11950 1700
-	1    0    0    -1
-$EndComp
+	0    -1   -1   0
+$EndComp
+Text Label 11950 1200 0    60   ~ 0
+PWR
 $EndSCHEMATC

Commit message: Fix EE_CS
Parts:
- DA2: symbol TLV700XX -> TLV700xx
- DA3: symbol LD1117 -> LD1117-RESCUE-Glidertrack
- F1: symbol FUSE0R -> Fuse0R
- XL1: symbol USB_MINI_B -> USB_MINI_B-RESCUE-Glidertrack
Connections:
- net labels removed: EE_CK
Changed lines of the file:
@@
 EESchema Schematic File Version 2
+LIBS:Glidertrack-rescue
 LIBS:Connectors_kl
 LIBS:modules
@@
 LIBS:memory
 LIBS:Glidertrack-cache
-EELAYER 27 0
+EELAYER 25 0
 EELAYER END
 $Descr A3 16535 11693
@@
 $EndComp
 $Comp
-L USB_MINI_B XL1
+L USB_MINI_B-RESCUE-Glidertrack XL1
 U 1 1 5476152F
 P 1400 2000
@@
 SWCLK
 $Comp
-L TLV700XX DA2
+L TLV700xx DA2
 U 1 1 54761A87
 P 7000 9950
@@
 NoConn ~ 9200 3800
 $Comp
-L LD1117 DA3
+L LD1117-RESCUE-Glidertrack DA3
 U 1 1 5481EBBD
 P 4500 9950
@@
 	3650 9900 4200 9900
 $Comp
-L +VS #PWR027
+L +Vs #PWR027
 U 1 1 5481EC4D
 P 3650 9900
@@
 MOTOR_FLAG
 $Comp
-L FUSE0R F1
+L Fuse0R F1
 U 1 1 548204A9
 P 2100 8850
@@
 	1650 9750 1650 9550
 $Comp
-L +VS #PWR046
+L +Vs #PWR046
 U 1 1 54820F54
 P 1650 9550
@@
 EE_SCK
 Text Label 6550 2900 2    60   ~ 0
-EE_CK
+EE_CS
 Wire Wire Line
 	5050 2150 5250 2150
